Commit message: added performance environment

File: ai_race/sim_environment/urdf/camera_macro.xacro (robot description, xacro)
@@ -54,5 +54,5 @@
     </gazebo>
   </xacro:macro>
-    <xacro:macro name="camera_macro_640x480" params="parent prefix xyz">
+  <xacro:macro name="camera_macro_640x480" params="parent prefix xyz">
     <joint name="${prefix}_joint" type="fixed">
       <parent link="${parent}"/>
@@ -108,3 +108,58 @@
     </gazebo>
   </xacro:macro>
+  <xacro:macro name="camera_macro_perspective_720x480" params="parent prefix xyz x_rot y_rot z_rot">
+    <joint name="${prefix}_joint" type="fixed">
+      <parent link="${parent}"/>
+      <child  link="${prefix}_link"/>
+      <origin xyz="${xyz}" rpy="${radians(-90)} 0 ${radians(-90)}"/>
+      <!--<origin xyz="${xyz}" rpy="${radians(x_rot)} ${radians(y_rot)} ${radians(z_rot)}"/>-->
+    </joint>
+    <link name="${prefix}_link">
+      <visual>
+        <origin xyz="0 0 0" rpy="0 0 0" />
+        <geometry>
+          <box size="0.01 0.01 0.03" />
+        </geometry>
+        <material name="Green" />
+      </visual>
+    </link>
+    <gazebo reference="${prefix}_link">
+      <sensor type="camera" name="${prefix}">
+        <update_rate>10.0</update_rate>
+        <camera name="${prefix}">
+          <pose>0 0 0 ${radians(x_rot)} ${radians(y_rot)} ${radians(z_rot)}"</pose>
+          <!--<horizontal_fov>1.3962634</horizontal_fov>-->
+          <horizontal_fov>1.4</horizontal_fov>
+          <image>
+            <width>720</width>
+            <height>480</height>
+            <format>R8G8B8</format>
+          </image>
+          <clip>
+            <near>0.02</near><!--default 0.02-->
+            <far>50</far>
+          </clip>
+          <noise>
+            <type>gaussian</type>
+            <mean>0.0</mean>
+            <stddev>0.007</stddev>
+          </noise>
+        </camera>
+        <plugin name="camera_controller" filename="libgazebo_ros_camera.so">
+          <alwaysOn>true</alwaysOn>
+          <updateRate>0.0</updateRate>
+          <cameraName>${prefix}</cameraName>
+          <imageTopicName>image_raw</imageTopicName>
+          <cameraInfoTopicName>camera_info</cameraInfoTopicName>
+          <frameName>${prefix}_link</frameName>
+          <hackBaseline>0.0</hackBaseline>
+          <distortionK1>0.0</distortionK1>
+          <distortionK2>0.0</distortionK2>
+          <distortionK3>0.0</distortionK3>
+          <distortionT1>0.0</distortionT1>
+          <distortionT2>0.0</distortionT2>
+        </plugin>
+      </sensor>
+    </gazebo>
+  </xacro:macro>
 </robot>

File: ai_race/sim_environment/urdf/godeye.urdf.xacro (robot description, xacro)
@@ -34,4 +34,5 @@
   <gazebo reference="base_footprint">
     <turnGravityOff>false</turnGravityOff>
+    <static>true</static>
   </gazebo>
   <!-- BASE-LINK -->

File: ai_race/sim_environment/urdf/godeye_perspective.urdf.xacro (robot description, xacro)
@@ -1,14 +1,13 @@
 <?xml version="1.0"?>
-<robot name="surveillance_camera_base" xmlns:xacro="http://www.ros.org/wiki/xacro">
+<robot name="godeye_perspective_base" xmlns:xacro="http://www.ros.org/wiki/xacro">
   <!-- Included URDF/XACRO Files -->
   <xacro:include filename="$(find sim_environment)/urdf/camera_macro.xacro" />
-  <xacro:include filename="$(find sim_environment)/urdf/ir_sensor_macro.xacro" />
   <!-- PROPERTY LIST -->
   <!--All units in m-kg-s-radians unit system -->
   <property name="M_PI" value="3.1415926535897931" />
   <!-- Main Body-base -->
-  <property name="base_x_size" value="0.05" />
-  <property name="base_y_size" value="0.05" />
-  <property name="base_z_size" value="0.3" />
+  <property name="base_x_size" value="0.01" />
+  <property name="base_y_size" value="0.01" />
+  <property name="base_z_size" value="0.01" />
   <property name="base_mass" value="1000" /> <!-- in kg-->
   <!--Inertial macros for the box and cylinder. Units are kg*m^2-->
@@ -47,11 +46,4 @@
       <box_inertia  m="${base_mass}" x="${base_x_size}" y="${base_y_size}" z="${base_z_size}"/>
     </inertial>
-    <visual>
-      <origin xyz="0 0 0" rpy="0 0 ${-M_PI/2}" />
-      <geometry>
-        <box size="${base_x_size} ${base_y_size} ${base_z_size}"/>
-      </geometry>
-      <!--<material name="Yellow" />-->
-    </visual>
     <collision>
       <origin xyz="0 0 0" rpy="0 0 0 " />
@@ -63,14 +55,13 @@
   <gazebo reference="base_link">
     <!--<material>Gazebo/Yellow</material>-->
-    <turnGravityOff>false</turnGravityOff>
+    <turnGravityOff>true</turnGravityOff>
   </gazebo>
   <joint name="base_footprint_joint" type="fixed">
-    <origin xyz="0 0 0.02" rpy="0 0 0" />
+    <origin xyz="0 0 0" rpy="0 1.5708 0" />
     <parent link="base_footprint"/>
     <child link="base_link" />
   </joint>
   <!-- camera -->
-  <camera_macro parent="base_link" prefix="surveillance_camera" xyz="0.1 0.0 0.12"/>
-  <ir_sensor_macro parent="base_link" prefix="ir_sensor" xyz="0.1 0.0 -0.12"/>
+  <camera_macro_perspective_720x480 parent="base_link" prefix="godeye_camera_perspective" xyz="-1.5 0.0 0" x_rot="0" y_rot="-150" z_rot="-38"/>
   <gazebo>
     <plugin name="gazebo_ros_control" filename="libgazebo_ros_control.so" />

Commit message: added maps2

File: ai_race/sim_environment/urdf/camera_macro.xacro (robot description, xacro)
@@ -163,3 +163,58 @@
     </gazebo>
   </xacro:macro>
+  <xacro:macro name="camera_macro_perspective2_720x480" params="parent prefix xyz x_rot y_rot z_rot">
+    <joint name="${prefix}_joint" type="fixed">
+      <parent link="${parent}"/>
+      <child  link="${prefix}_link"/>
+      <origin xyz="${xyz}" rpy="${radians(-90)} 0 ${radians(-90)}"/>
+      <!--<origin xyz="${xyz}" rpy="${radians(x_rot)} ${radians(y_rot)} ${radians(z_rot)}"/>-->
+    </joint>
+    <link name="${prefix}_link">
+      <visual>
+        <origin xyz="0 0 0" rpy="0 0 0" />
+        <geometry>
+          <box size="0.01 0.01 0.03" />
+        </geometry>
+        <material name="Green" />
+      </visual>
+    </link>
+    <gazebo reference="${prefix}_link">
+      <sensor type="camera" name="${prefix}">
+        <update_rate>10.0</update_rate>
+        <camera name="${prefix}">
+          <pose>0 0 0 ${radians(x_rot)} ${radians(y_rot)} ${radians(z_rot)}"</pose>
+          <!--<horizontal_fov>1.3962634</horizontal_fov>-->
+          <horizontal_fov>0.9</horizontal_fov>
+          <image>
+            <width>720</width>
+            <height>480</height>
+            <format>R8G8B8</format>
+          </image>
+          <clip>
+            <near>0.02</near><!--default 0.02-->
+            <far>50</far>
+          </clip>
+          <noise>
+            <type>gaussian</type>
+            <mean>0.0</mean>
+            <stddev>0.007</stddev>
+          </noise>
+        </camera>
+        <plugin name="camera_controller" filename="libgazebo_ros_camera.so">
+          <alwaysOn>true</alwaysOn>
+          <updateRate>0.0</updateRate>
+          <cameraName>${prefix}</cameraName>
+          <imageTopicName>image_raw</imageTopicName>
+          <cameraInfoTopicName>camera_info</cameraInfoTopicName>
+          <frameName>${prefix}_link</frameName>
+          <hackBaseline>0.0</hackBaseline>
+          <distortionK1>0.0</distortionK1>
+          <distortionK2>0.0</distortionK2>
+          <distortionK3>0.0</distortionK3>
+          <distortionT1>0.0</distortionT1>
+          <distortionT2>0.0</distortionT2>
+        </plugin>
+      </sensor>
+    </gazebo>
+  </xacro:macro>
 </robot>
